Commit message: gazebo kinda works

File: install/ur5e_description/share/ur5e_description/urdf/robotiq_85_gripper.urdf.xacro (robot description, xacro)
@@ -11,10 +11,10 @@
             <visual>
                 <geometry>
-                    <mesh filename="file://$(find ur5e_description)/meshes/robotiq_85/visual/robotiq_85_base_link.dae"/>
-                </geometry>
-            </visual>
-            <collision>
-                <geometry>
-                    <mesh filename="file://$(find ur5e_description)/meshes/robotiq_85/collision/robotiq_85_base_link.stl"/>
+                    <mesh filename="package://ur5e_description/meshes/visual/robotiq_85_base_link.dae"/>
+                </geometry>
+            </visual>
+            <collision>
+                <geometry>
+                    <mesh filename="package://ur5e_description/meshes/collision/robotiq_85_base_link.stl"/>
                 </geometry>
             </collision>
@@ -45,10 +45,10 @@
             <visual>
                 <geometry>
-                    <mesh filename="file://$(find ur5e_description)/meshes/robotiq_85/visual/robotiq_85_knuckle_link.dae"/>
-                </geometry>
-            </visual>
-            <collision>
-                <geometry>
-                    <mesh filename="file://$(find ur5e_description)/meshes/robotiq_85/collision/robotiq_85_knuckle_link.stl"/>
+                    <mesh filename="package://ur5e_description/meshes/visual/robotiq_85_knuckle_link.dae"/>
+                </geometry>
+            </visual>
+            <collision>
+                <geometry>
+                    <mesh filename="package://ur5e_description/meshes/collision/robotiq_85_knuckle_link.stl"/>
                 </geometry>
             </collision>
@@ -67,10 +67,10 @@
             <visual>
                 <geometry>
-                    <mesh filename="file://$(find ur5e_description)/meshes/robotiq_85/visual/robotiq_85_knuckle_link.dae"/>
-                </geometry>
-            </visual>
-            <collision>
-                <geometry>
-                    <mesh filename="file://$(find ur5e_description)/meshes/robotiq_85/collision/robotiq_85_knuckle_link.stl"/>
+                    <mesh filename="package://ur5e_description/meshes/visual/robotiq_85_knuckle_link.dae"/>
+                </geometry>
+            </visual>
+            <collision>
+                <geometry>
+                    <mesh filename="package://ur5e_description/meshes/collision/robotiq_85_knuckle_link.stl"/>
                 </geometry>
             </collision>
@@ -99,10 +99,10 @@
             <visual>
                 <geometry>
-                    <mesh filename="file://$(find ur5e_description)/meshes/robotiq_85/visual/robotiq_85_finger_link.dae"/>
-                </geometry>
-            </visual>
-            <collision>
-                <geometry>
-                    <mesh filename="file://$(find ur5e_description)/meshes/robotiq_85/collision/robotiq_85_finger_link.stl"/>
+                    <mesh filename="package://ur5e_description/meshes/visual/robotiq_85_finger_link.dae"/>
+                </geometry>
+            </visual>
+            <collision>
+                <geometry>
+                    <mesh filename="package://ur5e_description/meshes/collision/robotiq_85_finger_link.stl"/>
                 </geometry>
             </collision>
@@ -118,10 +118,10 @@
             <visual>
                 <geometry>
-                    <mesh filename="file://$(find ur5e_description)/meshes/robotiq_85/visual/robotiq_85_finger_link.dae"/>
-                </geometry>
-            </visual>
-            <collision>
-                <geometry>
-                    <mesh filename="file://$(find ur5e_description)/meshes/robotiq_85/collision/robotiq_85_finger_link.stl"/>
+                    <mesh filename="package://ur5e_description/meshes/visual/robotiq_85_finger_link.dae"/>
+                </geometry>
+            </visual>
+            <collision>
+                <geometry>
+                    <mesh filename="package://ur5e_description/meshes/collision/robotiq_85_finger_link.stl"/>
                 </geometry>
             </collision>
@@ -153,10 +153,10 @@
             <visual>
                 <geometry>
-                    <mesh filename="file://$(find ur5e_description)/meshes/robotiq_85/visual/robotiq_85_inner_knuckle_link.dae"/>
-                </geometry>
-            </visual>
-            <collision>
-                <geometry>
-                    <mesh filename="file://$(find ur5e_description)/meshes/robotiq_85/collision/robotiq_85_inner_knuckle_link.stl"/>
+                    <mesh filename="package://ur5e_description/meshes/visual/robotiq_85_inner_knuckle_link.dae"/>
+                </geometry>
+            </visual>
+            <collision>
+                <geometry>
+                    <mesh filename="package://ur5e_description/meshes/collision/robotiq_85_inner_knuckle_link.stl"/>
                 </geometry>
             </collision>
@@ -172,10 +172,10 @@
             <visual>
                 <geometry>
-                    <mesh filename="file://$(find ur5e_description)/meshes/robotiq_85/visual/robotiq_85_inner_knuckle_link.dae"/>
-                </geometry>
-            </visual>
-            <collision>
-                <geometry>
-                    <mesh filename="file://$(find ur5e_description)/meshes/robotiq_85/collision/robotiq_85_inner_knuckle_link.stl"/>
+                    <mesh filename="package://ur5e_description/meshes/visual/robotiq_85_inner_knuckle_link.dae"/>
+                </geometry>
+            </visual>
+            <collision>
+                <geometry>
+                    <mesh filename="package://ur5e_description/meshes/collision/robotiq_85_inner_knuckle_link.stl"/>
                 </geometry>
             </collision>
@@ -207,10 +207,10 @@
             <visual>
                 <geometry>
-                    <mesh filename="file://$(find ur5e_description)/meshes/robotiq_85/visual/robotiq_85_finger_tip_link.dae"/>
-                </geometry>
-            </visual>
-            <collision>
-                <geometry>
-                    <mesh filename="file://$(find ur5e_description)/meshes/robotiq_85/collision/robotiq_85_finger_tip_link.stl"/>
+                    <mesh filename="package://ur5e_description/meshes/visual/robotiq_85_finger_tip_link.dae"/>
+                </geometry>
+            </visual>
+            <collision>
+                <geometry>
+                    <mesh filename="package://ur5e_description/meshes/collision/robotiq_85_finger_tip_link.stl"/>
                 </geometry>
             </collision>
@@ -226,10 +226,10 @@
             <visual>
                 <geometry>
-                    <mesh filename="file://$(find ur5e_description)/meshes/robotiq_85/visual/robotiq_85_finger_tip_link.dae"/>
-                </geometry>
-            </visual>
-            <collision>
-                <geometry>
-                    <mesh filename="file://$(find ur5e_description)/meshes/robotiq_85/collision/robotiq_85_finger_tip_link.stl"/>
+                    <mesh filename="package://ur5e_description/meshes/visual/robotiq_85_finger_tip_link.dae"/>
+                </geometry>
+            </visual>
+            <collision>
+                <geometry>
+                    <mesh filename="package://ur5e_description/meshes/collision/robotiq_85_finger_tip_link.stl"/>
                 </geometry>
             </collision>

File: install/ur5e_description/share/ur5e_description/urdf/ur_macro.xacro (robot description, xacro)
@@ -72,5 +72,5 @@
         <origin xyz="0 0 0" rpy="0 0 ${pi}"/>
         <geometry>
-	        <mesh filename="file://$(find ur5e_description)/meshes/ur5e/visual/base.dae"/>
+	        <mesh filename="file://$(find ur5e_description)/meshes/ur5e/visual/base.dae" scale="0.001 0.001 0.001" />
         </geometry>
       </visual>
@@ -78,5 +78,5 @@
         <origin xyz="0 0 0" rpy="0 0 ${pi}"/>
         <geometry>
-	        <mesh filename="file://$(find ur5e_description)/meshes/ur5e/collision/base.stl"/>
+	        <mesh filename="file://$(find ur5e_description)/meshes/ur5e/collision/base.stl" scale="0.001 0.001 0.001" />
         </geometry>
       </collision>
@@ -89,5 +89,5 @@
         <origin xyz="0 0 0" rpy="0 0 ${pi}"/>
         <geometry>
-          <mesh filename="file://$(find ur5e_description)/meshes/ur5e/visual/shoulder.dae"/>
+          <mesh filename="file://$(find ur5e_description)/meshes/realsense_camera/d455.stl" scale="0.001 0.001 0.001" />
         </geometry>
       </visual>
@@ -95,5 +95,5 @@
         <origin xyz="0 0 0" rpy="0 0 ${pi}"/>
         <geometry>
-          <mesh filename="file://$(find ur5e_description)/meshes/ur5e/collision/shoulder.stl"/>
+          <mesh filename="file://$(find ur5e_description)/meshes/realsense_camera/d455.stl" scale="0.001 0.001 0.001" />
         </geometry>
       </collision>
@@ -114,5 +114,5 @@
         <origin xyz="0 0 ${shoulder_offset}" rpy="${pi/2} 0 ${-pi/2}"/>
         <geometry>
-        <mesh filename="file://$(find ur5e_description)/meshes/ur5e/visual/upperarm.dae"/>
+        <mesh filename="file://$(find ur5e_description)/meshes/realsense_camera/d455.stl" scale="0.001 0.001 0.001" />
         </geometry>
       </visual>
@@ -120,5 +120,5 @@
         <origin xyz="0 0 ${shoulder_offset}" rpy="${pi/2} 0 ${-pi/2}"/>
         <geometry>
-	        <mesh filename="file://$(find ur5e_description)/meshes/ur5e/collision/upperarm.stl"/>
+	        <mesh filename="file://$(find ur5e_description)/meshes/realsense_camera/d455.stl" scale="0.001 0.001 0.001" />
         </geometry>
       </collision>
@@ -140,5 +140,5 @@
         <origin xyz="0 0 ${elbow_offset}" rpy="${pi/2} 0 ${-pi/2}"/>
         <geometry>
-	        <mesh filename="file://$(find ur5e_description)/meshes/ur5e/visual/forearm.dae"/>
+	        <mesh filename="file://$(find ur5e_description)/meshes/realsense_camera/d455.stl" scale="0.001 0.001 0.001" />
         </geometry>
       </visual>
@@ -146,5 +146,5 @@
         <origin xyz="0 0 ${elbow_offset}" rpy="${pi/2} 0 ${-pi/2}"/>
         <geometry>
-	        <mesh filename="file://$(find ur5e_description)/meshes/ur5e/collision/forearm.stl"/>
+	        <mesh filename="file://$(find ur5e_description)/meshes/realsense_camera/d455.stl" scale="0.001 0.001 0.001" />
         </geometry>
       </collision>
@@ -167,5 +167,5 @@
       	<origin xyz="0 0 ${visual_params}" rpy="${pi/2} 0 0"/>
         <geometry>
-	        <mesh filename="file://$(find ur5e_description)/meshes/ur5e/visual/wrist1.dae"/>
+	        <mesh filename="file://$(find ur5e_description)/meshes/realsense_camera/d455.stl" scale="0.001 0.001 0.001" />
         </geometry>
       </visual>
@@ -173,5 +173,5 @@
         <origin xyz="0 0 ${visual_params}" rpy="${pi/2} 0 0"/>
         <geometry>
-	        <mesh filename="file://$(find ur5e_description)/meshes/ur5e/collision/wrist1.stl"/>
+	        <mesh filename="file://$(find ur5e_description)/meshes/realsense_camera/d455.stl" scale="0.001 0.001 0.001" />
         </geometry>
       </collision>
@@ -194,5 +194,5 @@
         <origin xyz="0 0 ${visual_params}" rpy="0 0 0"/>
         <geometry>
-	        <mesh filename="file://$(find ur5e_description)/meshes/ur5e/visual/wrist2.dae"/>
+	        <mesh filename="file://$(find ur5e_description)/meshes/realsense_camera/d455.stl" scale="0.001 0.001 0.001" />
         </geometry>
       </visual>
@@ -200,5 +200,5 @@
         <origin xyz="0 0 ${visual_params}" rpy="0 0 0"/>
         <geometry>
-	        <mesh filename="file://$(find ur5e_description)/meshes/ur5e/collision/wrist2.stl"/>
+	        <mesh filename="file://$(find ur5e_description)/meshes/realsense_camera/d455.stl" scale="0.001 0.001 0.001" />
         </geometry>
       </collision>
@@ -221,5 +221,5 @@
         <origin xyz="0 0 ${visual_params}" rpy="${pi/2} 0 0"/>
         <geometry>
-	        <mesh filename="file://$(find ur5e_description)/meshes/ur5e/visual/wrist3.dae"/>
+	        <mesh filename="file://$(find ur5e_description)/meshes/realsense_camera/d455.stl" scale="0.001 0.001 0.001" />
         </geometry>
       </visual>
@@ -227,5 +227,5 @@
         <origin xyz="0 0 ${visual_params}" rpy="${pi/2} 0 0"/>
         <geometry>
-	        <mesh filename="file://$(find ur5e_description)/meshes/ur5e/collision/wrist3.stl"/>
+	        <mesh filename="file://$(find ur5e_description)/meshes/realsense_camera/d455.stl" scale="0.001 0.001 0.001" />
         </geometry>
       </collision>
