Commit message: fix gripper xacro

File: urdf/gripper/robotiq_85_gripper.urdf.xacro (robot description, xacro)
@@ -1,5 +1,6 @@
 <?xml version="1.0"?>
 <robot name="robotiq_85_gripper" xmlns:xacro="http://ros.org/wiki/xacro">
-    <xacro:include filename="$(find ur5e_description)/urdf/robotiq_85_gripper.transmission.xacro" />
+    <xacro:include filename="$(find ur5e_description)/urdf/gripper/robotiq_85_gripper.transmission.xacro" />
+    <xacro:arg name="prefix" default=""/>
     <xacro:macro name="robotiq_85_gripper" params="prefix parent *origin">
         <joint name="${prefix}robotiq_85_base_joint" type="fixed">
@@ -40,5 +41,5 @@
             <origin rpy="0.0 0.0 0.0" xyz="0.05490451627 -0.03060114443 0.0"/>
             <limit lower="-3.14" upper="3.14" velocity="100.0" effort="1000"/>
-            <mimic joint="${prefix}robotiq_85_left_knuckle_joint"/>
+           <mimic joint="${prefix}robotiq_85_left_knuckle_joint"/>
         </joint>
         <link name="${prefix}robotiq_85_left_knuckle_link">
@@ -90,4 +91,5 @@
             <child link="${prefix}robotiq_85_left_finger_link"/>
             <origin xyz="-0.00408552455 -0.03148604435 0.0" rpy="0 0 0" />
+            <mimic joint="${prefix}robotiq_85_left_knuckle_joint" multiplier="1"/>
         </joint>
         <joint name="${prefix}robotiq_85_right_finger_joint" type="continuous">
@@ -95,4 +97,5 @@
             <child link="${prefix}robotiq_85_right_finger_link"/>
             <origin xyz="-0.00408552455 -0.03148604435 0.0" rpy="0 0 0" />
+            <mimic joint="${prefix}robotiq_85_left_knuckle_joint" multiplier="1"/>
         </joint>
         <link name="${prefix}robotiq_85_left_finger_link">
@@ -140,5 +143,5 @@
             <origin xyz="0.06142 0.0127 0" rpy="${pi} 0.0 0.0" />
             <limit lower="-3.14" upper="3.14" velocity="100.0" effort="0.1"/>
-            <mimic joint="${prefix}robotiq_85_left_knuckle_joint" offset="0"/>
+           <mimic joint="${prefix}robotiq_85_left_knuckle_joint" offset="0"/>
         </joint>
         <joint name="${prefix}robotiq_85_right_inner_knuckle_joint" type="continuous">
@@ -148,5 +151,5 @@
             <origin xyz="0.06142 -0.0127 0" rpy="0 0 0"/>
             <limit lower="-3.14" upper="3.14" velocity="100.0" effort="0.1"/>
-            <mimic joint="${prefix}robotiq_85_left_knuckle_joint" offset="0"/>
+          <mimic joint="${prefix}robotiq_85_left_knuckle_joint" offset="0"/>
         </joint>
         <link name="${prefix}robotiq_85_left_inner_knuckle_link">
@@ -194,5 +197,5 @@
             <origin xyz="0.04303959807 -0.03759940821 0.0" rpy="0.0 0.0 0.0"/>
             <limit lower="-3.14" upper="3.14" velocity="100.0" effort="0.1"/>
-            <mimic joint="${prefix}robotiq_85_left_knuckle_joint" multiplier="-1"/>
+          <mimic joint="${prefix}robotiq_85_left_knuckle_joint" multiplier="-1"/>
         </joint>
         <joint name="${prefix}robotiq_85_right_finger_tip_joint" type="continuous">
@@ -202,5 +205,5 @@
             <origin rpy="0.0 0.0 0.0" xyz="0.04303959807 -0.03759940821  0.0"/>
             <limit lower="-3.14" upper="3.14" velocity="100.0" effort="0.1"/>
-            <mimic joint="${prefix}robotiq_85_left_knuckle_joint" multiplier="-1"/>
+          <mimic joint="${prefix}robotiq_85_left_knuckle_joint" multiplier="-1"/>
         </joint>
         <link name="${prefix}robotiq_85_left_finger_tip_link">

File: urdf/realsense/_d455.urdf.xacro (robot description, xacro)
@@ -21,6 +21,6 @@
 <robot name="sensor_d455" xmlns:xacro="http://ros.org/wiki/xacro">
   <!-- Includes -->
-  <xacro:include filename="$(find ur5e_description)/urdf/_materials.urdf.xacro" />
-  <xacro:include filename="$(find ur5e_description)/urdf/_usb_plug.urdf.xacro" />
+  <xacro:include filename="$(find ur5e_description)/urdf/realsense/_materials.urdf.xacro" />
+  <xacro:include filename="$(find ur5e_description)/urdf/realsense/_usb_plug.urdf.xacro" />
   <xacro:macro name="sensor_d455" params="parent *origin name:=camera use_nominal_extrinsics:=false">
     <xacro:arg name="add_plug" default="false" />

File: urdf/ur5e/ur_macro.xacro (robot description, xacro)
@@ -1,48 +1,7 @@
 <?xml version="1.0"?>
 <robot xmlns:xacro="http://wiki.ros.org/xacro">
-  <!--
-    Base UR robot series xacro macro.
-    NOTE this is NOT a URDF. It cannot directly be loaded by consumers
-    expecting a flattened '.urdf' file. See the top-level '.xacro' for that
-    (but note that .xacro must still be processed by the xacro command).
-    This file models the base kinematic chain of a UR robot, which then gets
-    parameterised by various configuration files to convert it into a UR3(e),
-    UR5(e), UR10(e) or UR16e.
-    NOTE the default kinematic parameters (i.e., link lengths, frame locations,
-    offsets, etc) do not correspond to any particular robot. They are defaults
-    only. There WILL be non-zero offsets between the Forward Kinematics results
-    in TF (i.e., robot_state_publisher) and the values reported by the Teach
-    Pendant.
-    For accurate (and robot-specific) transforms, the 'kinematics_parameters_file'
-    parameter MUST point to a .yaml file containing the appropriate values for
-    the targeted robot.
-    If using the UniversalRobots/Universal_Robots_ROS_Driver, follow the steps
-    described in the readme of that repository to extract the kinematic
-    calibration from the controller and generate the required .yaml file.
-    Main author of the migration to yaml configs Ludovic Delval.
-    Contributors to previous versions (in no particular order)
-     - Denis Stogl
-     - Lovro Ivanov
-     - Felix Messmer
-     - Kelsey Hawkins
-     - Wim Meeussen
-     - Shaun Edwards
-     - Nadia Hammoudeh Garcia
-     - Dave Hershberger
-     - G. vd. Hoorn
-     - Philip Long
-     - Dave Coleman
-     - Miguel Prada
-     - Mathias Luedtke
-     - Marcel Schnirring
-     - Felix von Drigalski
-     - Felix Exner
-     - Jimmy Da Silva
-     - Ajit Krisshna N L
-     - Muhammad Asif Rana
-  -->
-  <xacro:include filename="$(find ur5e_description)/urdf/inc/ur_common.xacro" />
-  <xacro:include filename="$(find ur5e_description)/urdf/robotiq_85_gripper.urdf.xacro"/>
-  <xacro:include filename="$(find ur5e_description)/urdf/_d455.urdf.xacro" />
+  <xacro:include filename="$(find ur5e_description)/urdf/ur5e/inc/ur_common.xacro" />
+  <xacro:include filename="$(find ur5e_description)/urdf/gripper/robotiq_85_gripper.urdf.xacro"/>
+  <xacro:include filename="$(find ur5e_description)/urdf/realsense/_d455.urdf.xacro" />
   <xacro:macro name="ur_robot" params="
     name
@@ -253,9 +212,4 @@
       <parent link="${tf_prefix}base_link" />
       <child link="${tf_prefix}base_link_inertia" />
-      <!-- 'base_link' is REP-103 aligned (so X+ forward), while the internal
-           frames of the robot/controller have X+ pointing backwards.
-           Use the joint between 'base_link' and 'base_link_inertia' (a dummy
-           link/frame) to introduce the necessary rotation over Z (of pi rad).
-      -->
       <origin xyz="0 0 0" rpy="0 0 ${pi}" />
     </joint>

Commit message: 1 dof gripper

File: urdf/gripper/robotiq_85_gripper.urdf.xacro (robot description, xacro)
@@ -87,15 +87,13 @@
             </inertial>
         </link>
-        <joint name="${prefix}robotiq_85_left_finger_joint" type="continuous">
+        <joint name="${prefix}robotiq_85_left_finger_joint" type="fixed">
             <parent link="${prefix}robotiq_85_left_knuckle_link"/>
             <child link="${prefix}robotiq_85_left_finger_link"/>
             <origin xyz="-0.00408552455 -0.03148604435 0.0" rpy="0 0 0" />
-            <mimic joint="${prefix}robotiq_85_left_knuckle_joint" multiplier="1"/>
-        </joint>
-        <joint name="${prefix}robotiq_85_right_finger_joint" type="continuous">
+        </joint>
+        <joint name="${prefix}robotiq_85_right_finger_joint" type="fixed">
             <parent link="${prefix}robotiq_85_right_knuckle_link"/>
             <child link="${prefix}robotiq_85_right_finger_link"/>
             <origin xyz="-0.00408552455 -0.03148604435 0.0" rpy="0 0 0" />
-            <mimic joint="${prefix}robotiq_85_left_knuckle_joint" multiplier="1"/>
         </joint>
         <link name="${prefix}robotiq_85_left_finger_link">
