Commit message: fix gz sim physics

File: urdf/ur5e/ur.urdf.xacro (robot description, xacro)
@@ -1,5 +1,5 @@
 <?xml version="1.0"?>
 <robot xmlns:xacro="http://www.ros.org/wiki/xacro" name="ur">
-  <!-- Define los argumentos dentro del <robot> -->
+  <!-- Define los argumentos -->
   <xacro:arg name="name" default="ur"/>
   <xacro:arg name="ur_type" default="ur5e"/>
@@ -14,7 +14,9 @@
   <xacro:arg name="safety_k_position" default="20"/>
   <xacro:arg name="force_abs_paths" default="false"/>
-  <!-- Importa el macro principal -->
+  <!-- Incluye el xacro del robot -->
   <xacro:include filename="$(find ur5e_description)/urdf/ur5e/ur_macro.xacro"/>
-  <!-- Crea un link fijo al mundo -->
+  <!-- Incluye solo el archivo de macros de la garra -->
+  <xacro:include filename="$(find robotiq_description)/urdf/robotiq_2f_85_macro.urdf.xacro"/>
+  <!-- Link del mundo -->
   <link name="world" />
   <!-- Instancia el robot -->
@@ -33,3 +35,11 @@
     <origin xyz="0 0 0" rpy="0 0 0" />
   </xacro:ur_robot>
+  <!-- Instancia la garra y la une al link final 'tool0' -->
+  <xacro:robotiq_gripper
+      name="RobotiqGripperHardwareInterface"
+      prefix="gripper_"
+      parent="tool0"
+      use_fake_hardware="true">
+    <origin xyz="0 0 0" rpy="-1.57 0 -1.57"/>
+  </xacro:robotiq_gripper>
 </robot>

File: urdf/ur5e/ur_macro.xacro (robot description, xacro)
@@ -2,6 +2,4 @@
 <robot xmlns:xacro="http://wiki.ros.org/xacro">
   <xacro:include filename="$(find ur5e_description)/urdf/ur5e/inc/ur_common.xacro" />
-  <xacro:include filename="$(find ur5e_description)/urdf/gripper/robotiq_85_gripper.urdf.xacro"/>
-  <xacro:include filename="$(find ur5e_description)/urdf/realsense/_d455.urdf.xacro" />
   <xacro:macro name="ur_robot" params="
     name
@@ -319,8 +317,4 @@
       <origin xyz="0 0 0" rpy="0 ${-pi/2.0} ${-pi/2.0}" />
     </joint>
-    <!-- 🔹 Instanciamos la garra usando directamente el archivo URDF.XACRO -->
-    <xacro:robotiq_85_gripper prefix="gripper_" parent="${tf_prefix}flange">
-      <origin xyz="0 0 0" rpy="0 0 0"/>
-    </xacro:robotiq_85_gripper>
     <!-- ROS-Industrial 'tool0' frame - redefinido en la garra -->
     <link name="${tf_prefix}tool0"/>
@@ -330,12 +324,4 @@
       <child link="${tf_prefix}tool0"/>
     </joint>
-    <!-- Después de definir el chain principal y antes de cerrar el macro 'ur_robot' -->
-    <xacro:sensor_d455
-      parent="${tf_prefix}wrist_3_link"
-      name="camera_d455"
-      use_nominal_extrinsics="true">
-      <!-- Ajusta la posición y orientación de la cámara respecto a wrist_2_link -->
-      <origin xyz="0.0 -0.05 -0.06" rpy="0 -1.5708 1.5708"/>
-    </xacro:sensor_d455>
   </xacro:macro>
 </robot>
